File: trinity-devices-controller_24V/trinity-devices-controller_24V.kicad_pcb (KiCad board)
At the start: 4 copper layers, 90 x 70 mm, 145 parts, among them IC2 MCP2562, J1 xh2pin, J10 xh2pin, J16 xh2pin, J17 xh2pin, J18 xh2pin, J19 xh2pin, J2 xh2pin, J3 Conn_01x01_Pin, J4 Conn_01x01_Pin, J5 Conn_01x04, J6 Conn_01x04, J7 Conn_01x04_Pin, J8 Conn_01x04, J9 xh2pin, Q1 IRFML8244TRPBFTR, Q10 IRFML8244TRPBFTR, Q11 IRFML8244TRPBFTR, Q2 IRFML8244TRPBFTR, Q5 IRFML8244TRPBFTR, Q6 IRFML8244TRPBFTR, Q8 IRFML8244TRPBFTR, Q9 IRFML8244TRPBFTR, SW1 SW_Push, U1 TLP293-4, U2 NJW4132U2-B, U3 STM32G431K8Tx, U4 NJM12888F33, U5 TLP293-4, U6 NJM7812SDL1, U7 NJW4132U2-B

Commit message: FETをIRFML8244TRPbFからSSM6K819Rに変更
Parts:
- Q1, Q10, Q11, Q2, Q5, Q6, Q8, Q9: value IRFML8244TRPBFTR -> SSM6K819R; footprint Package_TO_SOT_SMD:SOT-23 -> 0Ikedalibrary:TSOP6F
- moved Q1 0.45 mm to (24.1, 21.9), turned to 0 degrees
- moved Q6 0.40 mm to (24.4, 50.6), turned to 0 degrees
- moved Q5 0.39 mm to (24.4, 42.0), turned to 0 degrees
- moved D3 0.30 mm to (23.3, 46.6)
- moved D1 0.25 mm to (23.3, 26.4)
- moved D4 0.25 mm to (23.3, 55.1)
- moved R22 0.25 mm to (25.3, 54.1)
- moved R23 0.25 mm to (26.9, 54.1)
- moved R5 0.20 mm to (23.9, 29.4)
- moved Q11 0.15 mm to (51.2, 39.0), turned to 180 degrees
- moved R6 0.15 mm to (23.9, 39.5)
- moved Q8 0.15 mm to (51.2, 31.4), turned to 180 degrees
- moved D2 0.14 mm to (23.4, 36.6)
- moved R3 0.10 mm to (25.3, 25.6)
- turned Q10 to 180 degrees
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Connections:
- Q1 pad 1: Net-(Q1-G) -> OUT1
- Q1 pad 2: GND -> OUT1
- Q1 pad 3: OUT1 -> Net-(Q1-G)
- Q10 pad 1: Net-(Q10-G) -> OUT7
- Q10 pad 2: GND -> OUT7
- Q10 pad 3: OUT7 -> Net-(Q10-G)
- Q11 pad 1: Net-(Q11-G) -> OUT8
- Q11 pad 2: GND -> OUT8
- Q11 pad 3: OUT8 -> Net-(Q11-G)
- Q2 pad 1: Net-(Q2-G) -> OUT2
- Q2 pad 2: GND -> OUT2
- Q2 pad 3: OUT2 -> Net-(Q2-G)
- Q5 pad 1: Net-(Q5-G) -> OUT3
- Q5 pad 2: GND -> OUT3
- Q5 pad 3: OUT3 -> Net-(Q5-G)
- Q6 pad 1: Net-(Q6-G) -> OUT4
- Q6 pad 2: GND -> OUT4
- Q6 pad 3: OUT4 -> Net-(Q6-G)
- Q8 pad 1: Net-(Q8-G) -> OUT5
- Q8 pad 2: GND -> OUT5
- Q8 pad 3: OUT5 -> Net-(Q8-G)
- Q9 pad 1: Net-(Q9-G) -> OUT6
- Q9 pad 2: GND -> OUT6
- Q9 pad 3: OUT6 -> Net-(Q9-G)
Routing:
- net OUT2: track 7.42 -> 5.65 mm
- net Net-(R60-Pad1): track 17.6 -> 19.0 mm
- net OUT4: track 7.05 -> 5.77 mm
- net OUT3: track 7.05 -> 5.81 mm
- net Net-(R3-Pad1): track 21.4 -> 22.2 mm
- net Net-(Q5-G): track 3.25 -> 2.61 mm
- added copper zone on F.Cu, net OUT1
- added copper zone on F.Cu, net OUT2
- added copper zone on F.Cu, net OUT3
- added copper zone on F.Cu, net OUT4
- added copper zone on F.Cu, net OUT5
- added copper zone on F.Cu, net OUT6
- added copper zone on F.Cu, net OUT7
- added copper zone on F.Cu, net OUT8

Commit message: ビア、シルク完成　ガーバの生成
Parts:
- F1, F2: value Fuse -> SF-1206FP100-2; footprint Fuse:Fuse_0603_1608Metric -> Capacitor_SMD:C_1206_3216Metric_Pad1.33x1.80mm_HandSolder
- moved G*** 1.80 mm to (57.1, 19.9)
- moved F2 0.50 mm to (100.0, 71.6)
- moved F1 0.50 mm to (100.0, 67.7)
- moved Q10 0.15 mm to (34.9, 42.2)
Routing:
- net VCC_2: track 15.6 -> 17.3 mm
- net OUT6: track 17.5 -> 18.3 mm
- net 24V_1: track 174.0 -> 173.4 mm
- net GND: vias 195 -> 290
