File: trinity-devices-controller_24V/trinity-devices-controller_24V.kicad_sch (KiCad schematic)
At the start: 140 parts, among them IC2 MCP2562, J1 xh2pin, J10 xh2pin, J16 xh2pin, J17 xh2pin, J18 xh2pin, J19 xh2pin, J2 xh2pin, J3 Conn_01x01_Pin, J4 Conn_01x01_Pin, J5 Conn_01x04, J6 Conn_01x04, J7 Conn_01x04_Pin, J8 Conn_01x04, J9 xh2pin, Q1 IRFML8244TRPBFTR, Q10 IRFML8244TRPBFTR, Q11 IRFML8244TRPBFTR, Q2 IRFML8244TRPBFTR, Q5 IRFML8244TRPBFTR, Q6 IRFML8244TRPBFTR, Q8 IRFML8244TRPBFTR, Q9 IRFML8244TRPBFTR, SW1 SW_Push, U1 TLP293-4, U2 NJW4132U2-B, U3 STM32G431K8Tx, U4 NJM12888F33, U5 TLP293-4, U6 NJM7812SDL1, U7 NJW4132U2-B

Commit message: FETをIRFML8244TRPbFからSSM6K819Rに変更
Parts:
- Q1, Q10, Q11, Q2, Q5, Q6, Q8, Q9: value IRFML8244TRPBFTR -> SSM6K819R; footprint Package_TO_SOT_SMD:SOT-23 -> 0Ikedalibrary:TSOP6F
Connections:
- net GND: now also Q1.4 (S), Q10.4 (S), Q11.4 (S), Q2.4 (S), Q5.4 (S), Q6.4 (S), Q8.4 (S), Q9.4 (S); no longer Q1.2 (S), Q10.2 (S), Q11.2 (S), Q2.2 (S), Q5.2 (S), Q6.2 (S), Q8.2 (S), Q9.2 (S)
- net OUT1: now also Q1.1 (D), Q1.2 (D), Q1.5 (D), Q1.6 (D); no longer Q1.3 (D)
- net OUT2: now also Q2.1 (D), Q2.2 (D), Q2.5 (D), Q2.6 (D); no longer Q2.3 (D)
- net OUT3: now also Q5.1 (D), Q5.2 (D), Q5.5 (D), Q5.6 (D); no longer Q5.3 (D)
- net OUT4: now also Q6.1 (D), Q6.2 (D), Q6.5 (D), Q6.6 (D); no longer Q6.3 (D)
- net OUT5: now also Q8.1 (D), Q8.2 (D), Q8.5 (D), Q8.6 (D); no longer Q8.3 (D)
- net OUT6: now also Q9.1 (D), Q9.2 (D), Q9.5 (D), Q9.6 (D); no longer Q9.3 (D)
- net OUT7: now also Q10.1 (D), Q10.2 (D), Q10.5 (D), Q10.6 (D); no longer Q10.3 (D)
- net OUT8: now also Q11.1 (D), Q11.2 (D), Q11.5 (D), Q11.6 (D); no longer Q11.3 (D)
- net at R3.2: now also Q1.3 (G); no longer Q1.1 (G)
- net at R63.2: now also Q11.3 (G); no longer Q11.1 (G)
- net at R19.2: now also Q5.3 (G); no longer Q5.1 (G)
- net at R62.2: now also Q10.3 (G); no longer Q10.1 (G)
- net at R22.2: now also Q6.3 (G); no longer Q6.1 (G)
- net at R61.2: now also Q9.3 (G); no longer Q9.1 (G)
- net at R60.2: now also Q8.3 (G); no longer Q8.1 (G)
- net at R4.2: now also Q2.3 (G); no longer Q2.1 (G)

Commit message: ビア、シルク完成　ガーバの生成
Parts:
- F1, F2: value Fuse -> SF-1206FP100-2; footprint Fuse:Fuse_0603_1608Metric -> Capacitor_SMD:C_1206_3216Metric_Pad1.33x1.80mm_HandSolder
Other:
- moved on the sheet: C10, C12, C13, C6, C7, C8, C9, D10, F1, L2, R10, R11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
